Commit message: Fully functioning UGV AgileX Scout 2.0 autonomous navigation  on gazebo at Aarhus Airport

File: simulation/src/runway_description/urdf/ugv.urdf.xacro (robot description, xacro)
@@ -1,172 +1,5 @@
 <?xml version="1.0"?>
-<robot xmlns:xacro="http://www.ros.org/wiki/xacro" name="runway_ugv">
-  <link name="base_footprint"/>
-  <joint name="base_footprint_joint" type="fixed">
-    <parent link="base_footprint"/>
-    <child link="base_link"/>
-    <origin xyz="0 0 0.15" rpy="0 0 0"/>
-  </joint>
-  <link name="base_link">
-    <visual>
-      <geometry>
-        <box size="0.8 0.5 0.2"/>
-      </geometry>
-      <material name="dark_gray">
-        <color rgba="0.2 0.2 0.2 1.0"/>
-      </material>
-    </visual>
-    <collision>
-      <geometry>
-        <box size="0.8 0.5 0.2"/>
-      </geometry>
-    </collision>
-    <inertial>
-      <mass value="25.0"/>
-      <inertia ixx="0.604" ixy="0.0" ixz="0.0" iyy="1.416" iyz="0.0" izz="1.854"/>
-    </inertial>
-  </link>
-  <xacro:macro name="wheel" params="prefix x_reflect y_reflect">
-    <link name="${prefix}_wheel_link">
-      <visual>
-        <origin xyz="0 0 0" rpy="${pi/2} 0 0"/>
-        <geometry>
-          <cylinder radius="0.15" length="0.08"/>
-        </geometry>
-        <material name="orange">
-          <color rgba="0.9 0.4 0.0 1.0"/>
-        </material>
-      </visual>
-      <collision>
-        <origin xyz="0 0 0" rpy="${pi/2} 0 0"/>
-        <geometry>
-          <cylinder radius="0.15" length="0.08"/>
-        </geometry>
-      </collision>
-      <inertial>
-        <mass value="2.5"/>
-        <inertia ixx="0.0154" ixy="0.0" ixz="0.0" iyy="0.0154" iyz="0.0" izz="0.0281"/>
-      </inertial>
-    </link>
-    <joint name="${prefix}_wheel_joint" type="continuous">
-      <parent link="base_link"/>
-      <child link="${prefix}_wheel_link"/>
-      <origin xyz="${x_reflect*0.25} ${y_reflect*0.29} 0.0" rpy="0 0 0"/>
-      <axis xyz="0 1 0"/>
-    </joint>
-    <gazebo reference="${prefix}_wheel_link">
-      <mu1>1.0</mu1>
-      <mu2>1.0</mu2>
-    </gazebo>
-  </xacro:macro>
-  <xacro:wheel prefix="front_left"  x_reflect="1"  y_reflect="1" />
-  <xacro:wheel prefix="front_right" x_reflect="1"  y_reflect="-1" />
-  <xacro:wheel prefix="rear_left"   x_reflect="-1" y_reflect="1" />
-  <xacro:wheel prefix="rear_right"  x_reflect="-1" y_reflect="-1" />
-  <link name="lidar_link">
-    <visual>
-      <geometry>
-        <cylinder radius="0.05" length="0.06"/>
-      </geometry>
-      <material name="blue">
-        <color rgba="0.1 0.1 0.8 1.0"/>
-      </material>
-    </visual>
-    <collision>
-      <geometry>
-        <cylinder radius="0.05" length="0.06"/>
-      </geometry>
-    </collision>
-  </link>
-  <joint name="lidar_joint" type="fixed">
-    <parent link="base_link"/>
-    <child link="lidar_link"/>
-    <origin xyz="0.2 0.0 0.13" rpy="0 0 0"/>
-  </joint>
-  <link name="camera_link">
-    <visual>
-      <geometry>
-        <box size="0.04 0.12 0.04"/>
-      </geometry>
-      <material name="red">
-        <color rgba="0.8 0.1 0.1 1.0"/>
-      </material>
-    </visual>
-    <collision>
-      <geometry>
-        <box size="0.04 0.12 0.04"/>
-      </geometry>
-    </collision>
-  </link>
-  <joint name="camera_joint" type="fixed">
-    <parent link="base_link"/>
-    <child link="camera_link"/>
-    <origin xyz="0.4 0.0 0.05" rpy="0 0 0"/>
-  </joint>
-  <link name="camera_optical_frame"/>
-  <joint name="camera_optical_joint" type="fixed">
-    <parent link="camera_link"/>
-    <child link="camera_optical_frame"/>
-    <origin xyz="0 0 0" rpy="${-pi/2} 0 ${-pi/2}"/>
-  </joint>
-  <gazebo>
-    <plugin filename="gz-sim-diff-drive-system" name="gz::sim::systems::DiffDrive">
-      <left_joint>front_left_wheel_joint</left_joint>
-      <left_joint>rear_left_wheel_joint</left_joint>
-      <right_joint>front_right_wheel_joint</right_joint>
-      <right_joint>rear_right_wheel_joint</right_joint>
-      <wheel_separation>0.58</wheel_separation>
-      <wheel_radius>0.15</wheel_radius>
-      <odom_publish_frequency>50</odom_publish_frequency>
-      <topic>/cmd_vel</topic>
-      <odom_topic>/odom</odom_topic>
-      <tf_topic>/tf</tf_topic>
-      <frame_id>odom</frame_id>
-      <child_frame_id>base_footprint</child_frame_id>
-    </plugin>
-  </gazebo>
-  <gazebo reference="lidar_link">
-    <sensor name="lidar" type="gpu_lidar">
-      <gz_frame_id>lidar_link</gz_frame_id>
-      <topic>/scan</topic>
-      <update_rate>10</update_rate>
-      <ray>
-        <scan>
-          <horizontal>
-            <samples>360</samples>
-            <resolution>1</resolution>
-            <min_angle>-3.14159</min_angle>
-            <max_angle>3.14159</max_angle>
-          </horizontal>
-        </scan>
-        <range>
-          <min>0.12</min>
-          <max>20.0</max>
-          <resolution>0.01</resolution>
-        </range>
-      </ray>
-      <always_on>1</always_on>
-      <visualize>true</visualize>
-    </sensor>
-  </gazebo>
-  <gazebo reference="camera_link">
-    <sensor name="camera" type="camera">
-      <gz_frame_id>camera_optical_frame</gz_frame_id>
-      <topic>/camera/image_raw</topic>
-      <update_rate>30</update_rate>
-      <camera>
-        <horizontal_fov>1.3962634</horizontal_fov>
-        <image>
-          <width>1280</width>
-          <height>720</height>
-          <format>R8G8B8</format>
-        </image>
-        <clip>
-          <near>0.1</near>
-          <far>100</far>
-        </clip>
-      </camera>
-      <always_on>1</always_on>
-      <visualize>true</visualize>
-    </sensor>
-  </gazebo>
+<robot name="runway_ugv" xmlns:xacro="http://ros.org/wiki/xacro">
+    <!-- Main UGV description based on Scout v2 chassis with Runway Inspection Payload -->
+    <xacro:include filename="$(find runway_description)/urdf/scout_v2.xacro" />
 </robot>
