Commit message: added communication feat and UI assets

File: simulation/src/runway_description/urdf/scout_v2.xacro (robot description, xacro)
@@ -30,11 +30,8 @@
             </geometry>
         </collision>
-        <collision>
-            <origin xyz="0 0 ${base_z_size/6}" rpy="0 0 0" />
-            <geometry>
-                <box size="${base_x_size/6} ${base_y_size*1.65} ${base_z_size/3}"/>
-            </geometry>
-        </collision>
-    </link>
+    </link>
+    <gazebo reference="base_link">
+        <self_collide>false</self_collide>
+    </gazebo>
     <link name="base_footprint"/>
     <joint name="base_footprint_joint" type="fixed">
@@ -183,5 +180,5 @@
             <right_joint>front_right_wheel</right_joint>
             <right_joint>rear_right_wheel</right_joint>
-            <wheel_separation>${track}</wheel_separation>
+            <wheel_separation>0.68</wheel_separation>
             <wheel_radius>${wheel_radius}</wheel_radius>
             <max_linear_acceleration>4.0</max_linear_acceleration>

File: simulation/src/runway_description/urdf/scout_wheel_type1.xacro (robot description, xacro)
@@ -6,5 +6,5 @@
                 <mass value="3.0" />
                 <origin xyz="0 0 0" />
-                <inertia ixx="0.7171" ixy="0" ixz="0" iyy="0.1361" iyz="0" izz="0.7171" />
+                <inertia ixx="0.0237" ixy="0" ixz="0" iyy="0.0406" iyz="0" izz="0.0237" />
             </inertial>
             <visual>
@@ -26,12 +26,14 @@
             <xacro:insert_block name="joint_pose"/>
             <axis xyz="${axis_xyz}" rpy="0 0 0" />
+            <dynamics damping="0.01" friction="0.01"/>
         </joint>
         <gazebo reference="${wheel_prefix}_wheel_link">
-            <mu1 value="1.0"/>
-            <mu2 value="0.1"/>
-            <fdir1 value="1 0 0"/>
-            <kp value="500000.0" />
-            <kd value="10.0" />
-            <minDepth>0.005</minDepth>
+            <mu1>1.2</mu1>
+            <mu2>0.2</mu2>
+            <kp>1000000.0</kp>
+            <kd>100.0</kd>
+            <minDepth>0.001</minDepth>
+            <maxVel>0.1</maxVel>
+            <fdir1>1 0 0</fdir1>
         </gazebo>
     </xacro:macro>

File: simulation/src/runway_description/urdf/scout_wheel_type2.xacro (robot description, xacro)
@@ -6,5 +6,5 @@
                 <mass value="3.0" />
                 <origin xyz="0 0 0" />
-                <inertia ixx="0.7171" ixy="0" ixz="0" iyy="0.1361" iyz="0" izz="0.7171" />
+                <inertia ixx="0.0237" ixy="0" ixz="0" iyy="0.0406" iyz="0" izz="0.0237" />
             </inertial>
             <visual>
@@ -26,12 +26,14 @@
             <xacro:insert_block name="joint_pose"/>
             <axis xyz="${axis_xyz}" rpy="0 0 0" />
+            <dynamics damping="0.01" friction="0.01"/>
         </joint>
         <gazebo reference="${wheel_prefix}_wheel_link">
-            <mu1 value="1.0"/>
-            <mu2 value="0.1"/>
-            <fdir1 value="1 0 0"/>
-            <kp value="500000.0" />
-            <kd value="10.0" />
-            <minDepth>0.005</minDepth>
+            <mu1>1.2</mu1>
+            <mu2>0.2</mu2>
+            <kp>1000000.0</kp>
+            <kd>100.0</kd>
+            <minDepth>0.001</minDepth>
+            <maxVel>0.1</maxVel>
+            <fdir1>1 0 0</fdir1>
         </gazebo>
     </xacro:macro>

Commit message: feat: Implement comprehensive ROS 2 simulation with Rviz2, Gazebo, Nav2, and DDS-based inter-vehicle communication.

File: simulation/src/runway_description/urdf/scout_v2.xacro (robot description, xacro)
@@ -125,4 +125,48 @@
         <parent link="camera_link" />
         <child link="camera_optical_link" />
+    </joint>
+    <!-- IMU Sensor Mount (Industrial 9-DOF IMU centered near CG) -->
+    <link name="imu_link">
+        <inertial>
+            <mass value="0.02" />
+            <origin xyz="0 0 0" />
+            <inertia ixx="0.000005" ixy="0" ixz="0" iyy="0.000005" iyz="0" izz="0.000005" />
+        </inertial>
+        <visual>
+            <origin xyz="0 0 0" rpy="0 0 0" />
+            <geometry>
+                <box size="0.03 0.03 0.015" />
+            </geometry>
+            <material name="orange">
+                <color rgba="1.0 0.5 0.0 1.0" />
+            </material>
+        </visual>
+    </link>
+    <joint name="imu_joint" type="fixed">
+        <origin xyz="0.0 0.0 0.08" rpy="0 0 0" />
+        <parent link="base_link" />
+        <child link="imu_link" />
+    </joint>
+    <!-- RTK-GNSS Antenna Mount (Elevated mast above chassis) -->
+    <link name="gps_link">
+        <inertial>
+            <mass value="0.05" />
+            <origin xyz="0 0 0" />
+            <inertia ixx="0.00001" ixy="0" ixz="0" iyy="0.00001" iyz="0" izz="0.00001" />
+        </inertial>
+        <visual>
+            <origin xyz="0 0 0" rpy="0 0 0" />
+            <geometry>
+                <cylinder length="0.03" radius="0.04" />
+            </geometry>
+            <material name="white">
+                <color rgba="0.95 0.95 0.95 1.0" />
+            </material>
+        </visual>
+    </link>
+    <joint name="gps_joint" type="fixed">
+        <origin xyz="-0.15 0.0 0.22" rpy="0 0 0" />
+        <parent link="base_link" />
+        <child link="gps_link" />
     </joint>
     <!-- Gazebo Sensor & Actuation Plugins -->
@@ -174,4 +218,32 @@
         </sensor>
     </gazebo>
+    <gazebo reference="imu_link">
+        <sensor name="imu_sensor" type="imu">
+            <always_on>true</always_on>
+            <update_rate>50</update_rate>
+            <topic>/imu/data</topic>
+            <gz_frame_id>imu_link</gz_frame_id>
+            <imu>
+                <angular_velocity>
+                    <x><noise type="gaussian"><mean>0.0</mean><stddev>0.0002</stddev></noise></x>
+                    <y><noise type="gaussian"><mean>0.0</mean><stddev>0.0002</stddev></noise></y>
+                    <z><noise type="gaussian"><mean>0.0</mean><stddev>0.0002</stddev></noise></z>
+                </angular_velocity>
+                <linear_acceleration>
+                    <x><noise type="gaussian"><mean>0.0</mean><stddev>0.01</stddev></noise></x>
+                    <y><noise type="gaussian"><mean>0.0</mean><stddev>0.01</stddev></noise></y>
+                    <z><noise type="gaussian"><mean>0.0</mean><stddev>0.01</stddev></noise></z>
+                </linear_acceleration>
+            </imu>
+        </sensor>
+    </gazebo>
+    <gazebo reference="gps_link">
+        <sensor name="navsat_sensor" type="navsat">
+            <always_on>true</always_on>
+            <update_rate>10</update_rate>
+            <topic>/gps/fix</topic>
+            <gz_frame_id>gps_link</gz_frame_id>
+        </sensor>
+    </gazebo>
     <gazebo>
         <plugin filename="gz-sim-diff-drive-system" name="gz::sim::systems::DiffDrive">
@@ -195,5 +267,4 @@
             <child_frame_id>base_footprint</child_frame_id>
             <odom_publish_frequency>50</odom_publish_frequency>
-            <tf_topic>/tf</tf_topic>
         </plugin>
         <plugin filename="gz-sim-joint-state-publisher-system" name="gz::sim::systems::JointStatePublisher">
